File: KiCAD/PC-8001MEMSD.sch (KiCad schematic (older format))
At the start: 17 parts, among them U1 74LS08, U2 74LS139, U3 74LS32, U4 74LS32, U5 74LS00, U6 74LS74, U7 CY7C199

Commit message: 回路図修正、logisimデータ追加
Parts:
- renumbered C1 to C?, C2 to C?, C3 to C?, C4 to C?, C5 to C?, C6 to C?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
Connections:
- net labels added: MODE-A0, MODE-A1
- net labels removed: D1, MODE-D0, MODE-D1
